File: PCB/fpga-power.kicad_sch (KiCad schematic)
At the start: 59 parts, among them U1 XC7Z020-1CLG400C

Commit message: added audio_start
Parts:
- renumbered C4 to C127, C10 to C128, C5 to C132, C11 to C133, C6 to C136, C12 to C137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
