File: PCB/fpga-power.kicad_sch (KiCad schematic)
At the start: 59 parts, among them U1 XC7Z020-1CLG400C

Commit message: [+] pre-BOM push
Parts:
- removed unit 4 of U1
- removed unit 3 of U1
- removed unit 1 of U1
- removed unit 2 of U1
- added C701, C702, C703, C705, C707, C709: 0.1uF 16V, symbol Device:C_Small
- added C704, C706, C708, C710: 0.01uF 25V, symbol Device:C_Small
- added J701: PH_4x1V_2.54mm, symbol Connector:Conn_01x04_Socket
- added J702: Conn_01x04_Socket, symbol Connector:Conn_01x04_Socket
- added R701, R702, R703: 80.6 1%, symbol Device:R_Small
- added R704, R708: 10k 1%, symbol Device:R_Small
- added R705: 200 1%, symbol Device:R_Small
- added R706, R707: 49.9 5%, symbol Device:R_Small
- added R709, R710, R713, R714, R715, R716, R720, R721: 1k 1%, symbol Device:R_Small
- added R711, R712, R717, R718, R719, R722, R723: 20k 1%, symbol Device:R_Small
- added R724: 0, symbol Device:R_Small
- added R725: 40.2 5%, symbol Device:R_Small
- added S701: SWITCH, symbol Simulation_SPICE:SWITCH
- added SW501: SW_DIP_x01, symbol Switch:SW_DIP_x01
- added U501: S25FL128SAGMFI000, SO3016_SPA, symbol S25FL128SAGMFI000:S25FL128SAGMFI000
- added U701: XC7Z020-1CLG400C, CLG400_ZYNQ-7000_XIL, symbol 2025-02-08_12-13-43:XC7Z020-1CLG400C
- added U702: NC7WZ07P6X, SC-88/SC70-6/SOT-363_419B-02_ONS, symbol 2025-02-19_13-54-14:NC7WZ07P6X
- added Y701: DSC1121CE5-050.0000, DSC1121CE50500000, symbol DSC1121CE5-050_0000:DSC1121CE5-050.0000
Connections:
- net GND: now also C701.2, C702.2, C703.2, C704.2, C705.2, C706.2, C707.2, C708.2, C709.2, C710.2, J701.2 (Pin_2), R702.1, R710.1, R714.2, R716.2, R718.1, R719.1, R720.2, R721.2, S701.2 (N-), U702.2 (GND), Y701.3 (GND)
- net VCC1V5: now also R701.1, R713.1
- net VCC1V8: now also R704.1, R715.1
- net VCC3V3: now also C701.1, C702.1, J701.4 (Pin_4), J702.1 (Pin_1), R708.1, R709.2, R717.1, U702.5 (VCC), Y701.1 (EN), Y701.6 (VDD)
- net VREF0V9: now reaches U1.E11 (PS_MIO_VREF_501)
- net VREF0V9: now also C707.1, C708.1, C709.1, C710.1, R715.2, R716.1
- net DDR3_VREF: now reaches U1.H6 (PS_DDR_VREF0_502)
- net DDR3_VREF: now also U1.P6 (PS_DDR_VREF1_502), C703.1, C704.1, C705.1, C706.1, R713.2, R714.1
- new net: R705.2, S701.1 (N+)
- new net: J701.1 (Pin_1), R709.1, R711.1
- new net: J702.2 (Pin_2), R720.1, R722.1
- new net: J702.4 (Pin_4), R721.1, R723.1
- new net: J701.3 (Pin_3), R710.2, R712.1
- new net: R724.1, U701.A5 (PS_MIO6_500)
- new net: R725.2, U701.D14 (PS_MIO40_501)
- new net: R706.1, R707.1, Y701.4 (OUT)
- new net AR_RST: R708.2, U701.D9 (PS_MIO12_500), U702.4 (Y2)
- new net DDR3_D0: U701.C3 (PS_DDR_DQ0_502)
- new net DDR3_D1: U701.B3 (PS_DDR_DQ1_502)
- new net DDR3_D10: U701.G3 (PS_DDR_DQ10_502)
- new net DDR3_D11: U701.H3 (PS_DDR_DQ11_502)
- new net DDR3_D12: U701.J3 (PS_DDR_DQ12_502)
- new net DDR3_D13: U701.H2 (PS_DDR_DQ13_502)
- new net DDR3_D14: U701.H1 (PS_DDR_DQ14_502)
- new net DDR3_D15: U701.J1 (PS_DDR_DQ15_502)
- new net DDR3_D2: U701.A2 (PS_DDR_DQ2_502)
- new net DDR3_D3: U701.A4 (PS_DDR_DQ3_502)
- new net DDR3_D4: U701.D3 (PS_DDR_DQ4_502)
- new net DDR3_D5: U701.D1 (PS_DDR_DQ5_502)
- new net DDR3_D6: U701.C1 (PS_DDR_DQ6_502)
- new net DDR3_D7: U701.E1 (PS_DDR_DQ7_502)
- new net DDR3_D8: U701.E2 (PS_DDR_DQ8_502)
- new net DDR3_D9: U701.E3 (PS_DDR_DQ9_502)
- new net DDR_VRN: R701.2, U701.G5 (PS_DDR_VRN_502)
- new net DDR_VRP: R702.2, U701.H5 (PS_DDR_VRP_502)
- new net ETH_CLK: R707.2
- new net ETH_INT_B: U701.E9 (PS_MIO10_500)
- new net ETH_MDC: U701.C10 (PS_MIO52_501)
- new net ETH_RST_B: U701.B5 (PS_MIO9_500)
- new net ETH_RXCK: U701.B17 (PS_MIO22_501)
- new net ETH_RXCTL: U701.D13 (PS_MIO27_501)
- new net ETH_RXD0: U701.D11 (PS_MIO23_501)
- new net ETH_RXD1: U701.A16 (PS_MIO24_501), U701.C11 (PS_MIO53_501)
- new net ETH_RXD2: U701.F15 (PS_MIO25_501)
- new net ETH_RXD3: U701.A15 (PS_MIO26_501)
- new net ETH_TXCK: U701.A19 (PS_MIO16_501)
- new net ETH_TXCTL: U701.F14 (PS_MIO21_501)
- new net ETH_TXD0: U701.E14 (PS_MIO17_501)
- new net ETH_TXD1: U701.B18 (PS_MIO18_501)
- new net ETH_TXD2: U701.D10 (PS_MIO19_501)
- new net ETH_TXD3: U701.A17 (PS_MIO20_501)
- new net HDMI_TX_SCL: U701.B13 (PS_MIO50_501)
- new net HDMI_TX_SDA: U701.B9 (PS_MIO51_501)
- new net MEM_ADD0: U701.N2 (PS_DDR_A0_502)
- new net MEM_ADD1: U701.K2 (PS_DDR_A1_502)
- new net MEM_ADD10: U701.F5 (PS_DDR_A10_502)
- new net MEM_ADD11: U701.G4 (PS_DDR_A11_502)
- new net MEM_ADD12: U701.E4 (PS_DDR_A12_502)
- new net MEM_ADD13: U701.D4 (PS_DDR_A13_502)
- new net MEM_ADD14: U701.F4 (PS_DDR_A14_502)
- new net MEM_ADD2: U701.M3 (PS_DDR_A2_502)
- new net MEM_ADD3: U701.K3 (PS_DDR_A3_502)
- new net MEM_ADD4: U701.M4 (PS_DDR_A4_502)
- new net MEM_ADD5: U701.L1 (PS_DDR_A5_502)
- new net MEM_ADD6: U701.L4 (PS_DDR_A6_502)
- new net MEM_ADD7: U701.K4 (PS_DDR_A7_502)
- new net MEM_ADD8: U701.K1 (PS_DDR_A8_502)
- new net MEM_ADD9: U701.J4 (PS_DDR_A9_502)
- new net MEM_BANK0: U701.L5 (PS_DDR_BA0_502)
- new net MEM_BANK1: U701.R4 (PS_DDR_BA1_502)
- new net MEM_BANK2: U701.J5 (PS_DDR_BA2_502)
- new net MEM_CAS#: U701.P5 (PS_DDR_CAS_B_502)
- new net MEM_CLK0_N: R703.1, U701.M2 (PS_DDR_CKN_502)
- new net MEM_CLK0_P: R703.2, U701.L2 (PS_DDR_CKP_502)
- new net MEM_DM0: U701.A1 (PS_DDR_DM0_502), U701.F1 (PS_DDR_DM1_502)
- new net MEM_DQS0_N: U701.B2 (PS_DDR_DQS_N0_502)
- new net MEM_DQS0_P: U701.C2 (PS_DDR_DQS_P0_502)
- new net MEM_DQS1_N: U701.F2 (PS_DDR_DQS_N1_502)
- new net MEM_DQS1_P: U701.G2 (PS_DDR_DQS_P1_502)
- new net MEM_MA0_CKE0: U701.N3 (PS_DDR_CKE_502)
- new net MEM_MA0_CS_L0: U701.N1 (PS_DDR_CS_B_502)
- new net MEM_MA0_ODT0: U701.N5 (PS_DDR_ODT_502)
- new net MEM_RAS#: U701.P4 (PS_DDR_RAS_B_502)
- new net MEM_RESET#: U701.B4 (PS_DDR_DRST_B_502)
- new net MEM_WE#: U701.M5 (PS_DDR_WE_B_502)
- new net OTG_CLK: U701.A11 (PS_MIO36_501)
- new net OTG_DATA0: U701.A14 (PS_MIO32_501)
- new net OTG_DATA1: U701.D15 (PS_MIO33_501)
- new net OTG_DATA2: U701.A12 (PS_MIO34_501)
- new net OTG_DATA3: U701.F12 (PS_MIO35_501)
- new net OTG_DATA4: U701.C16 (PS_MIO28_501)
- new net OTG_DATA5: U701.A10 (PS_MIO37_501)
- new net OTG_DATA6: U701.E13 (PS_MIO38_501)
- new net OTG_DATA7: U701.C18 (PS_MIO39_501)
- new net OTG_DIR: U701.C13 (PS_MIO29_501)
- new net OTG_NXT: U701.E16 (PS_MIO31_501)
- new net OTG_OC: U701.C6 (PS_MIO11_500)
- new net OTG_RESETN: U701.D16 (PS_MIO46_501)
- new net OTG_STP: U701.C15 (PS_MIO30_501)
- new net PG_ALL: U701.C7 (PS_POR_B_500)
- new net PS_CLK: R706.2, U701.E7 (PS_CLK_500)
- new net PS_RST: R704.2, R705.1, U701.B10 (PS_SRST_B_501), U702.3 (A2)
- new net SD_CCLK: R725.1
- new net SD_CD: U701.B14 (PS_MIO47_501)
- new net SD_CMD: U701.C17 (PS_MIO41_501)
- new net SD_D0: U701.E12 (PS_MIO42_501)
- new net SD_D1: U701.A9 (PS_MIO43_501)
- new net SD_D2: U701.F13 (PS_MIO44_501)
- new net SD_D3: U701.B15 (PS_MIO45_501)
- new net SPI_CS: U701.A7 (PS_MIO1_500)
- new net SPI_DQ0/MODE3: R722.2, U701.B8 (PS_MIO2_500)
- new net SPI_DQ1/MODE1: R719.2, U701.D6 (PS_MIO3_500)
- new net SPI_DQ2/MODE2: R712.2, U701.B7 (PS_MIO4_500)
- new net SPI_DQ3/MODE0: R711.2, U701.A6 (PS_MIO5_500)
- new net SPI_SCK/MODE4: R723.2, R724.2
- new net SPI_SCLK_FB/VCFG1: R717.2, U701.D5 (PS_MIO8_500)
- new net UART_RXD_OUT: U701.C8 (PS_MIO15_500)
- new net UART_TXD_IN: U701.C5 (PS_MIO14_500)
- new net VCFG0: R718.2, U701.D8 (PS_MIO7_500)
- no-connect marks 0 -> 27
Other:
- moved on the sheet: C69, C70, C71, C72, C73, C74, C75, C76, C77, C78, C79, C80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

Commit message: some part done
Parts:
- removed Y701: DSC1121CE5-050.0000, DSC1121CE50500000, symbol DSC1121CE5-050_0000:DSC1121CE5-050.0000
- added C645, C646: 0.1uF 16V, Capacitor_SMD:C_0805_2012Metric, symbol Device:C_Small
- added C647: 0.1uF 16V 0805, Capacitor_SMD:C_0805_2012Metric, symbol Device:C_Small
- added J601: Conn_01x04_Socket, symbol Connector:Conn_01x04_Socket
- added J602: Conn_01x02_Socket, symbol Connector:Conn_01x02_Socket
- added LED601: SML-LX1206SRC-TR, ul_SML-LX1206SRC-TR:LED_3P2X1P5_LUM, symbol 2025-02-15_04-53-13:SML-LX1206SRC-TR
- added R601, R602: 220 1%, Resistor_SMD:R_0805_2012Metric, symbol Device:R_Small_US
- added R603, R604, R605, R606: 100 5%, Resistor_SMD:R_0805_2012Metric, symbol Device:R_Small_US
- added R607, R608: 140 1%, Resistor_SMD:R_0805_2012Metric, symbol Device:R_Small_US
- added R609, R610: 4.7K 5%, Resistor_SMD:R_0805_2012Metric, symbol Device:R_Small_US
- added Y602: DSC1121CE5-050.0000, DSC1121CE5:DSC1121CE50500000, symbol DSC1121CE5-050_0000:DSC1121CE5-050.0000
- C1, C15, C9: footprint (none) -> Capacitor_SMD:C_1206_3216Metric
- C10, C11, C12, C13, C14, C16, C17, C2, C3, C4, C5, C6, C7, C8: footprint (none) -> Capacitor_SMD:C_0805_2012Metric
- C601: renamed from C82; footprint (none) -> Capacitor_SMD:C_1206_3216Metric
- C602: renamed from C88; footprint (none) -> Capacitor_SMD:C_1206_3216Metric
- C603: renamed from C94; footprint (none) -> Capacitor_SMD:C_1206_3216Metric
- C604: renamed from C83; footprint (none) -> Capacitor_SMD:C_0805_2012Metric
- C605: renamed from C89; footprint (none) -> Capacitor_SMD:C_0805_2012Metric
- C606: renamed from C95; footprint (none) -> Capacitor_SMD:C_0805_2012Metric
- C607: renamed from C84; footprint (none) -> Capacitor_SMD:C_0805_2012Metric
- C608: renamed from C90; footprint (none) -> Capacitor_SMD:C_0805_2012Metric
- C609: renamed from C96; footprint (none) -> Capacitor_SMD:C_0805_2012Metric
- C610: renamed from C91; footprint (none) -> Capacitor_SMD:C_0805_2012Metric
- C611: renamed from C92; footprint (none) -> Capacitor_SMD:C_0805_2012Metric
- C612: renamed from C93; footprint (none) -> Capacitor_SMD:C_0805_2012Metric
- C613: renamed from C106; footprint (none) -> Capacitor_SMD:C_1206_3216Metric
- C614: renamed from C112; footprint (none) -> Capacitor_SMD:C_1206_3216Metric
- C615: renamed from C100; footprint (none) -> Capacitor_SMD:C_1206_3216Metric
- C616: renamed from C107; footprint (none) -> Capacitor_SMD:C_0805_2012Metric
- C617: renamed from C113; footprint (none) -> Capacitor_SMD:C_0805_2012Metric
- C618: renamed from C101; footprint (none) -> Capacitor_SMD:C_0805_2012Metric
- C621: renamed from C108; footprint (none) -> Capacitor_SMD:C_0805_2012Metric
- C622: renamed from C114; footprint (none) -> Capacitor_SMD:C_0805_2012Metric
- C623: renamed from C102; footprint (none) -> Capacitor_SMD:C_0805_2012Metric
- C626: renamed from C109; footprint (none) -> Capacitor_SMD:C_0805_2012Metric
- C627: renamed from C115; footprint (none) -> Capacitor_SMD:C_0805_2012Metric
- C631: renamed from C110; footprint (none) -> Capacitor_SMD:C_0805_2012Metric
- C635: renamed from C111; footprint (none) -> Capacitor_SMD:C_0805_2012Metric
- C638: renamed from C85; footprint (none) -> Capacitor_SMD:C_0805_2012Metric
- C642: renamed from C86; footprint (none) -> Capacitor_SMD:C_0805_2012Metric
- C648: renamed from C70; footprint (none) -> Capacitor_SMD:C_0805_2012Metric
- C649: renamed from C71; footprint (none) -> Capacitor_SMD:C_0805_2012Metric
- C650: renamed from C72; footprint (none) -> Capacitor_SMD:C_0805_2012Metric
- C651: renamed from C76; footprint (none) -> Capacitor_SMD:C_0805_2012Metric
- C652: renamed from C73; footprint (none) -> Capacitor_SMD:C_0805_2012Metric
- C653: renamed from C77; footprint (none) -> Capacitor_SMD:C_0805_2012Metric
- C654: renamed from C74; footprint (none) -> Capacitor_SMD:C_0805_2012Metric
- C655: renamed from C69; footprint (none) -> Capacitor_SMD:C_0805_2012Metric
- C656: renamed from C78; footprint (none) -> Capacitor_SMD:C_1206_3216Metric
- C657: renamed from C75; footprint (none) -> Capacitor_SMD:C_1206_3216Metric
- C658: renamed from C79; footprint (none) -> Capacitor_SMD:C_1206_3216Metric
- C659: renamed from C80; footprint (none) -> Capacitor_SMD:C_0805_2012Metric
- C660: renamed from C81; footprint (none) -> Capacitor_SMD:C_0805_2012Metric
- C661: renamed from C701; footprint (none) -> Capacitor_SMD:C_0805_2012Metric
- C662: renamed from C702; footprint (none) -> Capacitor_SMD:C_0805_2012Metric
- C663: renamed from C703; footprint (none) -> Capacitor_SMD:C_0805_2012Metric
- C664: renamed from C704; footprint (none) -> Capacitor_SMD:C_0805_2012Metric
- C665: renamed from C705; footprint (none) -> Capacitor_SMD:C_0805_2012Metric
- C666: renamed from C706; footprint (none) -> Capacitor_SMD:C_0805_2012Metric
- C667: renamed from C707; footprint (none) -> Capacitor_SMD:C_0805_2012Metric
- C668: renamed from C708; footprint (none) -> Capacitor_SMD:C_0805_2012Metric
- C669: renamed from C709; footprint (none) -> Capacitor_SMD:C_0805_2012Metric
- C670: renamed from C710; footprint (none) -> Capacitor_SMD:C_0805_2012Metric
- FB1: footprint (none) -> Inductor_SMD:L_0603_1608Metric
- R611: renamed from R701; footprint (none) -> Resistor_SMD:R_0805_2012Metric
- R612: renamed from R702; footprint (none) -> Resistor_SMD:R_0805_2012Metric
- R613: renamed from R703; footprint (none) -> Resistor_SMD:R_0805_2012Metric
- R614: renamed from R704; footprint (none) -> Resistor_SMD:R_0805_2012Metric
- R615: renamed from R705; footprint (none) -> Resistor_SMD:R_0805_2012Metric
- R616: renamed from R706; footprint (none) -> Resistor_SMD:R_0805_2012Metric
- R617: renamed from R707; footprint (none) -> Resistor_SMD:R_0805_2012Metric
- R618: renamed from R708; footprint (none) -> Resistor_SMD:R_0805_2012Metric
- R619: renamed from R709; footprint (none) -> Resistor_SMD:R_0805_2012Metric
- R620: renamed from R710; footprint (none) -> Resistor_SMD:R_0805_2012Metric
- R621: renamed from R711; footprint (none) -> Resistor_SMD:R_0805_2012Metric
- R622: renamed from R712; footprint (none) -> Resistor_SMD:R_0805_2012Metric
- R623: renamed from R713; footprint (none) -> Resistor_SMD:R_0805_2012Metric
- R624: renamed from R714; footprint (none) -> Resistor_SMD:R_0805_2012Metric
- R625: renamed from R715; footprint (none) -> Resistor_SMD:R_0805_2012Metric
- R626: renamed from R716; footprint (none) -> Resistor_SMD:R_0805_2012Metric
- R627: renamed from R717; footprint (none) -> Resistor_SMD:R_0805_2012Metric
- R628: renamed from R718; footprint (none) -> Resistor_SMD:R_0805_2012Metric
- R629: renamed from R719; footprint (none) -> Resistor_SMD:R_0805_2012Metric
- R630: renamed from R720; footprint (none) -> Resistor_SMD:R_0805_2012Metric
- R631: renamed from R721; footprint (none) -> Resistor_SMD:R_0805_2012Metric
- R632: renamed from R722; footprint (none) -> Resistor_SMD:R_0805_2012Metric
- R633: renamed from R723; footprint (none) -> Resistor_SMD:R_0805_2012Metric
- R634: renamed from R724; footprint (none) -> Resistor_SMD:R_0805_2012Metric
- R635: renamed from R725; footprint (none) -> Resistor_SMD:R_0805_2012Metric
- U1: footprint ul_XC7Z020-1CLG400C:CLG400_ZYNQ-7000_XIL-L -> ul_XC7Z020-1CLG400C:CLG400_ZYNQ-7000_XIL
- U601: renamed from U701; footprint CLG400_ZYNQ-7000_XIL -> ul_XC7Z020-1CLG400C:CLG400_ZYNQ-7000_XIL
- U601: renamed from U1; footprint CLG400_ZYNQ-7000_XIL -> ul_XC7Z020-1CLG400C:CLG400_ZYNQ-7000_XIL
- U602: renamed from U501; footprint SO3016_SPA -> S25FL128SAGMFI000:SO3016_SPA
- renumbered J701 to J603, J702 to J604, S701 to S601, SW501 to SW601, U702 to U603
Connections:
- net GND: now also U1.L9 (VREFP_0), U601.F10 (RSVDGND), U601.J10 (GNDADC_0), U601.M10 (DXN_0), U601.M9 (DXP_0), U601.R20 (GND), U601.T13 (GND), U601.U16 (GND), U601.V19 (GND), U601.W12 (GND), U601.Y15 (GND), U602.10 (VSS), C645.2, C647.2, J602.2 (Pin_2), LED601.1, Y602.3 (GND)
- net SPI_CS: now also U602.7 (*CS), R610.1
- net SPI_DQ0/MODE3: now also U602.15 (SI/IO0)
- net SPI_DQ1/MODE1: now also U602.8 (SO/IO1)
- net SPI_DQ2/MODE2: now also U602.9 (*WP/IO2)
- net SPI_DQ3/MODE0: now also U602.1 (*HOLD/IO3)
- net SPI_SCK/MODE4: now also U602.16 (SCK)
- net VCC1V8: now also U601.J9 (VCCADC_0)
- net VCC3V3: now also U601.M6 (CFGBVS_0), U601.N6 (RSVDVCC3), U601.R6 (RSVDVCC2), U601.T6 (RSVDVCC1), U602.2 (VCC), C647.1, J602.1 (Pin_1), R601.2, R609.2, R610.2, Y602.1 (EN), Y602.6 (VDD)
- net TDI_USB/TDO_FPGA: now reaches U601.F6 (TDO_0)
- net TDI_USB/TDO_FPGA: now also R605.2
- net TCK: now reaches U601.F9 (TCK_0)
- net TCK: now also R606.2
- net TDO_USB/TDI_FPGA: now reaches U601.G6 (TDI_0)
- net TDO_USB/TDI_FPGA: now also R604.2
- net TMS: now reaches U601.J6 (TMS_0)
- net TMS: now also R603.2
- net at U601.K9 (VP_0): now also R608.1
- net at U601.L10 (VN_0): now also R607.1
- net PROGRAM_B: now reaches U601.L6 (PROGRAM_B_0)
- net INT_B_0: now reaches U601.R10 (INIT_B_0)
- net INT_B_0: now also R609.1
- net DONE_0: now reaches U601.R11 (DONE_0)
- net DONE_0: now also R601.1, R602.2
- net at R616.1, R617.1: now also Y602.4 (OUT)
- net XADCVREF: now reaches U1.K10 (VREFN_0)
- net XADCVREF: now also C645.1
- new net: LED601.2, R602.1
- new net: J601.3 (Pin_3), R605.1
- new net: J601.4 (Pin_4), R606.1
- new net: J601.2 (Pin_2), R604.1
- new net: J601.1 (Pin_1), R603.1
- new net XADC_V_N: C646.1, R607.2
- new net XADC_V_P: C646.2, R608.2
- no-connect marks 27 -> 29
Other:
- note added: "JTAG needs to be removed"
- moved on the sheet: C16, C17, C648, C649, C650, C651, C652, C653, C654, C655, C656, C657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
