File: PCB/fpga-power.kicad_sch (KiCad schematic)
At the start: 118 parts, among them J601 Conn_01x04_Socket, J602 Conn_01x02_Socket, J603 PH_4x1V_2.54mm, J604 Conn_01x04_Socket, SW601 SW_DIP_x01, U1 XC7Z020-1CLG400C, U601 XC7Z020-1CLG400C, U602 S25FL128SAGMFI000, U603 NC7WZ07P6X, Y602 DSC1121CE5-050.0000

Commit message: merge commit
Connections:
- net VCC1V5: no longer U1.G1 (VCCO_DDR_502), U1.H4 (VCCO_DDR_502), U1.L3 (VCCO_DDR_502), U1.U1 (VCCO_DDR_502)
- net VCC3V3: no longer U1.V14 (VCCO_34), U1.W17 (VCCO_34)
