File: PCB/gameboy.kicad_sch (KiCad schematic)
At the start: 0 parts

Commit message: Added headphoen audio
Changed lines of the file:
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@@
 	)
 	(sheet
-		(at 156.21 77.47)
+		(at 162.56 102.235)
 		(size 28.575 18.415)
 		(fields_autoplaced yes)
@@
 		)
 		(property "Sheetname" "SD card"
-			(at 156.21 76.7584 0)
+			(at 162.56 101.5234 0)
 			(effects
 				(font
@@
 		)
 		(property "Sheetfile" "sd.kicad_sch"
-			(at 156.21 96.4696 0)
+			(at 162.56 121.2346 0)
 			(effects
 				(font
