File: PCB/DDR.kicad_sch (KiCad schematic)
At the start: 22 parts, among them IC1 MT41K512M16HA-125__A

Commit message: some part done
Parts:
- C501: renamed from C28; footprint (none) -> Capacitor_SMD:C_0805_2012Metric
- C502: renamed from C53; footprint (none) -> Capacitor_SMD:C_0805_2012Metric
- C503: renamed from C54; footprint (none) -> Capacitor_SMD:C_0805_2012Metric
- C504: renamed from C66; footprint (none) -> Capacitor_SMD:C_0805_2012Metric
- C505: renamed from C55; footprint (none) -> Capacitor_SMD:C_0805_2012Metric
- C506: renamed from C67; footprint (none) -> Capacitor_SMD:C_0805_2012Metric
- C507: renamed from C56; footprint (none) -> Capacitor_SMD:C_0805_2012Metric
- C508: renamed from C68; footprint (none) -> Capacitor_SMD:C_0805_2012Metric
- C509: renamed from C57; footprint (none) -> Capacitor_SMD:C_0805_2012Metric
- C510: renamed from C62; footprint (none) -> Capacitor_SMD:C_0805_2012Metric
- C511: renamed from C58; footprint (none) -> Capacitor_SMD:C_0805_2012Metric
- C512: renamed from C63; footprint (none) -> Capacitor_SMD:C_0805_2012Metric
- C513: renamed from C59; footprint (none) -> Capacitor_SMD:C_0805_2012Metric
- C514: renamed from C64; footprint (none) -> Capacitor_SMD:C_0805_2012Metric
- C515: renamed from C60; footprint (none) -> Capacitor_SMD:C_0805_2012Metric
- C516: renamed from C65; footprint (none) -> Capacitor_SMD:C_0805_2012Metric
- C517: renamed from C61; footprint (none) -> Capacitor_SMD:C_0805_2012Metric
- IC501: renamed from IC1; footprint BGA96C80P9X16_900X1400X120 -> MT41K512M16HA:BGA96C80P9X16_900X1400X120
- R501: renamed from R40; footprint (none) -> Resistor_SMD:R_0805_2012Metric
- R502: renamed from R43; footprint (none) -> Resistor_SMD:R_0805_2012Metric
- R503: renamed from R41; footprint (none) -> Resistor_SMD:R_0805_2012Metric
- R504: renamed from R42; footprint (none) -> Resistor_SMD:R_0805_2012Metric
