File: PCB/sd.kicad_sch (KiCad schematic)
At the start: 9 parts, among them J301 Micro_SD_Card_Det1, J302 Micro_SD_Card_Det1, U301 TXS02612RTWR

Commit message: some part done
Parts:
- R301: renamed from R305; footprint (none) -> Resistor_SMD:R_0805_2012Metric
- R302: renamed from R303; footprint (none) -> Resistor_SMD:R_0805_2012Metric
- R303: renamed from R302; footprint (none) -> Resistor_SMD:R_0805_2012Metric
- R304: footprint (none) -> Resistor_SMD:R_0805_2012Metric
- R305: renamed from R301; footprint (none) -> Resistor_SMD:R_0805_2012Metric
Changed lines of the file:
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@@
 		(dnp no)
 		(fields_autoplaced yes)
-		(property "Reference" "#PWR0309"
+		(property "Reference" "#PWR0306"
 			(at 150.495 132.08 0)
 			(effects
@@
 			(project "gameboy"
 				(path "/bfbf29d7-ad29-43e7-b23f-5805508cd3f0/873f49b0-de10-4969-a045-ab304594bc32"
-					(reference "#PWR0309")
+					(reference "#PWR0306")
 					(unit 1)
 				)
@@
 		(dnp no)
 		(fields_autoplaced yes)
-		(property "Reference" "#PWR0310"
+		(property "Reference" "#PWR0302"
 			(at 103.505 69.85 0)
 			(effects
@@
 			(project "gameboy"
 				(path "/bfbf29d7-ad29-43e7-b23f-5805508cd3f0/873f49b0-de10-4969-a045-ab304594bc32"
-					(reference "#PWR0310")
+					(reference "#PWR0302")
 					(unit 1)
 				)
@@
 		(dnp no)
 		(fields_autoplaced yes)
-		(property "Reference" "#PWR0314"
+		(property "Reference" "#PWR0313"
 			(at 238.76 73.66 0)
 			(effects
@@
 			(project "gameboy"
 				(path "/bfbf29d7-ad29-43e7-b23f-5805508cd3f0/873f49b0-de10-4969-a045-ab304594bc32"
-					(reference "#PWR0314")
+					(reference "#PWR0313")
 					(unit 1)
 				)
@@
 		(dnp no)
 		(fields_autoplaced yes)
-		(property "Reference" "#PWR0307"
+		(property "Reference" "#PWR0311"
 			(at 190.5 68.58 0)
 			(effects
@@
 			(project "gameboy"
 				(path "/bfbf29d7-ad29-43e7-b23f-5805508cd3f0/873f49b0-de10-4969-a045-ab304594bc32"
-					(reference "#PWR0307")
+					(reference "#PWR0311")
 					(unit 1)
 				)
@@
 		(dnp no)
 		(fields_autoplaced yes)
-		(property "Reference" "#PWR0303"
+		(property "Reference" "#PWR0312"
 			(at 192.405 115.57 0)
 			(effects
@@
 			(project "gameboy"
 				(path "/bfbf29d7-ad29-43e7-b23f-5805508cd3f0/873f49b0-de10-4969-a045-ab304594bc32"
-					(reference "#PWR0303")
+					(reference "#PWR0312")
 					(unit 1)
 				)
@@
 		(dnp no)
 		(fields_autoplaced yes)
-		(property "Reference" "R305"
+		(property "Reference" "R301"
 			(at 112.395 64.77 90)
 			(effects
@@
 			)
 		)
-		(property "Footprint" ""
+		(property "Footprint" "Resistor_SMD:R_0805_2012Metric"
 			(at 112.395 69.85 0)
 			(effects
@@
 			(project "gameboy"
 				(path "/bfbf29d7-ad29-43e7-b23f-5805508cd3f0/873f49b0-de10-4969-a045-ab304594bc32"
-					(reference "R305")
+					(reference "R301")
 					(unit 1)
 				)
@@
 		(dnp no)
 		(fields_autoplaced yes)
-		(property "Reference" "#PWR0301"
+		(property "Reference" "#PWR0309"
 			(at 187.96 99.06 0)
 			(effects
@@
 			(project ""
 				(path "/bfbf29d7-ad29-43e7-b23f-5805508cd3f0/873f49b0-de10-4969-a045-ab304594bc32"
-					(reference "#PWR0301")
+					(reference "#PWR0309")
 					(unit 1)
 				)
@@
 		(dnp no)
 		(fields_autoplaced yes)
-		(property "Reference" "#PWR0312"
+		(property "Reference" "#PWR0301"
 			(at 102.87 71.12 0)
 			(effects
@@
 			(project "gameboy"
 				(path "/bfbf29d7-ad29-43e7-b23f-5805508cd3f0/873f49b0-de10-4969-a045-ab304594bc32"
-					(reference "#PWR0312")
+					(reference "#PWR0301")
 					(unit 1)
 				)
@@
 		(dnp no)
 		(fields_autoplaced yes)
-		(property "Reference" "#PWR0306"
+		(property "Reference" "#PWR0308"
 			(at 175.895 57.15 0)
 			(effects
@@
 			(project "gameboy"
 				(path "/bfbf29d7-ad29-43e7-b23f-5805508cd3f0/873f49b0-de10-4969-a045-ab304594bc32"
-					(reference "#PWR0306")
+					(reference "#PWR0308")
 					(unit 1)
 				)
@@
 		(dnp no)
 		(fields_autoplaced yes)
-		(property "Reference" "#PWR0311"
+		(property "Reference" "#PWR0305"
 			(at 146.685 62.23 0)
 			(effects
@@
 			(project "gameboy"
 				(path "/bfbf29d7-ad29-43e7-b23f-5805508cd3f0/873f49b0-de10-4969-a045-ab304594bc32"
-					(reference "#PWR0311")
+					(reference "#PWR0305")
 					(unit 1)
 				)
@@
 		(dnp no)
 		(fields_autoplaced yes)
-		(property "Reference" "#PWR0305"
+		(property "Reference" "#PWR0307"
 			(at 186.055 52.07 0)
 			(effects
@@
 			(project "gameboy"
 				(path "/bfbf29d7-ad29-43e7-b23f-5805508cd3f0/873f49b0-de10-4969-a045-ab304594bc32"
-					(reference "#PWR0305")
+					(reference "#PWR0307")
 					(unit 1)
 				)
@@
 		(dnp no)
 		(fields_autoplaced yes)
-		(property "Reference" "#PWR0313"
+		(property "Reference" "#PWR0314"
 			(at 240.665 120.65 0)
 			(effects
@@
 			(project "gameboy"
 				(path "/bfbf29d7-ad29-43e7-b23f-5805508cd3f0/873f49b0-de10-4969-a045-ab304594bc32"
-					(reference "#PWR0313")
+					(reference "#PWR0314")
 					(unit 1)
 				)
@@
 		(dnp no)
 		(fields_autoplaced yes)
-		(property "Reference" "#PWR0302"
+		(property "Reference" "#PWR0310"
 			(at 177.8 104.14 0)
 			(effects
@@
 			(project ""
 				(path "/bfbf29d7-ad29-43e7-b23f-5805508cd3f0/873f49b0-de10-4969-a045-ab304594bc32"
-					(reference "#PWR0302")
+					(reference "#PWR0310")
 					(unit 1)
 				)
@@
 		(dnp no)
 		(fields_autoplaced yes)
-		(property "Reference" "R303"
+		(property "Reference" "R302"
 			(at 192.405 69.2149 0)
 			(effects
@@
 			)
 		)
-		(property "Footprint" ""
+		(property "Footprint" "Resistor_SMD:R_0805_2012Metric"
 			(at 190.5 69.85 0)
 			(effects
@@
 			(project "gameboy"
 				(path "/bfbf29d7-ad29-43e7-b23f-5805508cd3f0/873f49b0-de10-4969-a045-ab304594bc32"
-					(reference "R303")
+					(reference "R302")
 					(unit 1)
 				)
@@
 		(dnp no)
 		(fields_autoplaced yes)
-		(property "Reference" "R301"
+		(property "Reference" "R305"
 			(at 194.945 109.22 90)
 			(effects
@@
 			)
 		)
-		(property "Footprint" ""
+		(property "Footprint" "Resistor_SMD:R_0805_2012Metric"
 			(at 194.945 114.3 0)
 			(effects
@@
 			(project "gameboy"
 				(path "/bfbf29d7-ad29-43e7-b23f-5805508cd3f0/873f49b0-de10-4969-a045-ab304594bc32"
-					(reference "R301")
+					(reference "R305")
 					(unit 1)
 				)
@@
 		(dnp no)
 		(fields_autoplaced yes)
-		(property "Reference" "#PWR0308"
+		(property "Reference" "#PWR0303"
 			(at 113.03 63.5 0)
 			(effects
@@
 			(project "gameboy"
 				(path "/bfbf29d7-ad29-43e7-b23f-5805508cd3f0/873f49b0-de10-4969-a045-ab304594bc32"
-					(reference "#PWR0308")
+					(reference "#PWR0303")
 					(unit 1)
 				)
@@
 		(dnp no)
 		(fields_autoplaced yes)
-		(property "Reference" "R302"
+		(property "Reference" "R303"
 			(at 194.31 116.2049 0)
 			(effects
@@
 			)
 		)
-		(property "Footprint" ""
+		(property "Footprint" "Resistor_SMD:R_0805_2012Metric"
 			(at 192.405 116.84 0)
 			(effects
@@
 			(project "gameboy"
 				(path "/bfbf29d7-ad29-43e7-b23f-5805508cd3f0/873f49b0-de10-4969-a045-ab304594bc32"
-					(reference "R302")
+					(reference "R303")
 					(unit 1)
 				)
@@
 			)
 		)
-		(property "Footprint" ""
+		(property "Footprint" "Resistor_SMD:R_0805_2012Metric"
 			(at 193.04 67.31 0)
 			(effects
