File: PCB/audio.kicad_sch (KiCad schematic)
At the start: 0 parts

Commit message: [+] add ZynqPCB
Parts:
- added C452, C454, C458: 0.1uF 16V, Capacitor_SMD:C_0805_2012Metric, symbol Device:C
- added C453, C455, C456, C457: 10uF 6.3V, Capacitor_SMD:C_0805_2012Metric, symbol Device:C
- added C459: 0.47uF 16V, Capacitor_SMD:C_0805_2012Metric, symbol Device:C
- added C460: 47p, Capacitor_SMD:C_0603_1608Metric, symbol Device:C
- added C461, C462: 100uF 25V, Capacitor_SMD:C_0805_2012Metric, symbol Device:C
- added C463, C464: 4700pF 50V, Capacitor_SMD:C_0603_1608Metric, symbol Device:C
- added C465, C466: 100pF 50V, Capacitor_SMD:C_0603_1608Metric, symbol Device:C
- added C467, C468: 10uF 25V, Capacitor_SMD:C_0805_2012Metric, symbol Device:C
- added C469, C470: 100pF 50V, Capacitor_SMD:C_0805_2012Metric, symbol Device:C
- added FB402, FB403, FB404, FB405: FerriteBead, Inductor_SMD:L_0805_2012Metric, symbol Device:FerriteBead
- added IC401: TS3A226AEYFFR, BGA9C40P3X3_126X136X62, symbol TS3A226AEYFFR:TS3A226AEYFFR
- added J402, J403: SJ-43515TS-SMT-TR, SJ-43515TS-SMT-TR:SJ43515TSSMTTR, symbol SJ-43515TS-SMT-TR:SJ-43515TS-SMT-TR
- added Q408: PMBT3904_215, SOT23_TO-236AB_NEX, symbol 2025-02-19_15-12-31:PMBT3904_215
- added R440, R441: 10K/X 1%, Resistor_SMD:R_0805_2012Metric, symbol Device:R
- added R442: 50, Resistor_SMD:R_0805_2012Metric, symbol Device:R
- added R443: 1M 1%, Resistor_SMD:R_0805_2012Metric, symbol Device:R
- added R444: 10k 1%, Resistor_SMD:R_0805_2012Metric, symbol Device:R
- added R445, R446: 1K 1%, Resistor_SMD:R_0603_1608Metric, symbol Device:R
- added U405: ADAU1761BCPZ, ADAU1761BCPZ:CP-32-4_ADI, symbol ADAU1761:ADAU1761BCPZ
Connections:
- new net: C469.1, FB404.2, J403.3 (RING_1)
- new net: C463.2, C467.1, R445.2
- new net: C470.1, FB405.2, J403.4 (RING_2)
- new net: C457.1, C458.1, U405.24 (DVDDOUT)
- new net: C464.1, C468.1, R446.2
- new net ADR0: U405.3 (ADDR0/CLATCH)
- new net ADR1: U405.30 (ADDR1/CDATA)
- new net AU_BCLK: U405.28 (BCLK/GPIO2)
- new net AU_DIN: U405.27 (DAC_SDATA/_GPIO0)
- new net AU_DOUT: U405.26 (ADC_SDATA/_GPIO1)
- new net AU_MCLK: R442.1
- new net AU_SCL: U405.32 (SCL/CCLK)
- new net AU_SDA: U405.31 (SDA/COUT)
- new net AU_WCLK: C460.1, U405.29 (LRCLK/GPIO3)
- new net CM: C452.1, C453.1, Q408.3, U405.10 (LINP), U405.11 (LINN), U405.12 (RINP), U405.13 (RINN), U405.7 (CM)
- new net FL_L: C461.1, U405.19 (RHP)
- new net FRONT L: C465.2, FB402.2, IC401.C2 (TIP), J402.2 (TIP)
- new net FRONT R: C466.2, FB403.2, J402.3 (RING_1), R444.1
- new net FRONT_L_C: C461.2, FB402.1
- new net FRONT_R_C: C462.2, FB403.1
- new net FR_L: C462.1, U405.20 (LHP)
- new net GND: C452.2, C453.2, C454.2, C455.2, C456.2, C457.2, C458.2, C459.2, C460.2, C463.1, C464.2, C465.1, C466.1, C469.2, C470.2, IC401.A2 (GNDB), IC401.B1 (MICP), IC401.B2 (GNDA), IC401.C3 (GND), J403.1 (SLEEVE), J403.2 (TIP), J403.5 (TIP_SWITCH), R440.2, R444.2, U405.22 (AGND), U405.25 (DGND), U405.9 (AGND)
- new net HP_EN: C459.1, IC401.C1 (EN), J402.5 (TIP_SWITCH), R443.2
- new net LAUX: C468.2, U405.6 (LAUX)
- new net LINE1_L_C: FB405.1, R446.1
- new net LINE1_R_C: FB404.1, R445.1
- new net MCLK1: R442.2, U405.2 (MCLK)
- new net MONOOUT: Q408.2, U405.21 (MONOOUT)
- new net Q19_1: Q408.1, R440.1, R441.1
- new net RAUX: C467.2, U405.14 (RAUX)
- new net RING2: IC401.A3 (RING2), J402.4 (RING_2)
- new net SLEEVE: IC401.B3 (SLEEVE), J402.1 (SLEEVE)
- new net VCC3V3: C454.1, C455.1, C456.1, IC401.A1 (VDD), R441.2, R443.1, U405.1 (IOVDD), U405.23 (AVDD), U405.8 (AVDD)
