File: PCB/peripherals.kicad_sch (KiCad schematic)
At the start: 0 parts

Commit message: [+] add ZynqPCB
Parts:
- added C201: 0.1uF 25V 0805, Capacitor_SMD:C_0805_2012Metric, symbol Device:C_Small
- added J201, J202: Conn_01x03_Socket, symbol Connector:Conn_01x03_Socket
- added R201, R202: 200 1%, Resistor_SMD:R_0805_2012Metric, symbol Device:R_Small_US
- added U201: ICM-20602, Package_LGA:LGA-16_3x3mm_P0.5mm_LayoutBorder3x5y, symbol Sensor_Motion:ICM-20602
Connections:
- new net: J202.2 (Pin_2), R201.2
- new net: J201.2 (Pin_2), R202.2
- new net: U201.10 (GND), U201.11 (GND), U201.12 (GND), U201.13 (GND), U201.15 (GND), U201.9 (GND)
- new net A20: U201.4 (SAO/SD0)
- new net B20: U201.3 (SDA/SDI)
- new net C20: U201.2 (SCL/SPC)
- new net GND: J201.3 (Pin_3), J202.3 (Pin_3)
- new net JA1_N: R201.1
- new net JA1_P: R202.1
- new net VCC3V3: J201.1 (Pin_1), J202.1 (Pin_1), U201.1 (VDDIO), U201.16 (VDD), U201.5 (~{CS})
Other:
- note added: "Touch buttons"
