File: PCB/Audio.kicad_sch (KiCad schematic)
At the start: 50 parts, among them J3 AUDIO JACK, Q1 IRLML2502, Q2 IRLML2502, Q3 IRLML2502, Q4 IRLML2502, Q5 IRLML2502, Q6 IRLML2502, U20 xc7z020clg484, U9 TLV320AIC3104

Commit message: [+] Layouting
Connections:
- net IR_RX: no longer names the net of U20.AA18 (IO_L12N_T1_MRCC_33)
- no-connect marks 46 -> 47
Changed lines of the file:
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@@
+	)
+	(no_connect
+		(at 50.8 74.93)
 	)
 	(no_connect
@@
 			(effects
 				(font
-					(size 1.27 1.27)
-				)
-				(hide yes)
-			)
-		)
-	)
-	(global_label "IR_RX"
-		(shape input)
-		(at 50.8 74.93 0)
-		(effects
-			(font
-				(size 1.524 1.524)
-			)
-			(justify left)
-		)
-		(property "Intersheetrefs" "${INTERSHEET_REFS}"
-			(at 50.8 74.93 0)
-			(effects
-				(font
