File: PCB/Audio.kicad_sch (KiCad schematic)
At the start: 50 parts, among them J3 AUDIO JACK, Q1 IRLML2502, Q2 IRLML2502, Q3 IRLML2502, Q4 IRLML2502, Q5 IRLML2502, Q6 IRLML2502, U20 xc7z020clg484, U9 TLV320AIC3104

Commit message: [+] routing done, need to fix minor errors.
Parts:
- gave numbers to parts that had none: 1
Changed lines of the file:
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@@
 		(on_board yes)
 		(dnp no)
-		(property "Reference" "#PWR?"
+		(property "Reference" "#PWR081"
 			(at 200.66 148.59 0)
 			(effects
@@
 		(instances
 			(project "DFTBoard"
-				(path "/0cf42e13-7c72-4f5f-898b-a3f851b94890/00000000-0000-0000-0000-000058508414"
-					(reference "#PWR?")
-					(unit 1)
-				)
 				(path "/0cf42e13-7c72-4f5f-898b-a3f851b94890/00000000-0000-0000-0000-000058508444"
 					(reference "#PWR081")
@@
 		(on_board yes)
 		(dnp no)
-		(property "Reference" "#PWR?"
+		(property "Reference" "#PWR082"
 			(at 200.66 175.26 0)
 			(effects
@@
 		(instances
 			(project "DFTBoard"
-				(path "/0cf42e13-7c72-4f5f-898b-a3f851b94890/00000000-0000-0000-0000-000058508414"
-					(reference "#PWR?")
-					(unit 1)
-				)
 				(path "/0cf42e13-7c72-4f5f-898b-a3f851b94890/00000000-0000-0000-0000-000058508444"
 					(reference "#PWR082")
@@
 		(on_board yes)
 		(dnp no)
-		(property "Reference" "GT?"
+		(property "Reference" "GT1"
 			(at 197.485 156.21 0)
 			(effects
@@
 		(instances
 			(project "DFTBoard"
-				(path "/0cf42e13-7c72-4f5f-898b-a3f851b94890/00000000-0000-0000-0000-000058508414"
-					(reference "GT?")
-					(unit 1)
-				)
 				(path "/0cf42e13-7c72-4f5f-898b-a3f851b94890/00000000-0000-0000-0000-000058508444"
 					(reference "GT1")
@@
 					(unit 1)
 				)
-				(path "/0cf42e13-7c72-4f5f-898b-a3f851b94890/00000000-0000-0000-0000-00005c7c62ae"
-					(reference "C?")
-					(unit 1)
-				)
 			)
 		)
@@
 					(unit 1)
 				)
-				(path "/0cf42e13-7c72-4f5f-898b-a3f851b94890/00000000-0000-0000-0000-00005c7c62ae"
-					(reference "#PWR?")
-					(unit 1)
-				)
 			)
 		)
@@
 					(unit 1)
 				)
-				(path "/0cf42e13-7c72-4f5f-898b-a3f851b94890/00000000-0000-0000-0000-00005c7c62ae"
-					(reference "#PWR?")
-					(unit 1)
-				)
 			)
 		)
@@
 					(unit 1)
 				)
-				(path "/0cf42e13-7c72-4f5f-898b-a3f851b94890/00000000-0000-0000-0000-00005c7c62ae"
-					(reference "Q?")
-					(unit 1)
-				)
 			)
 		)
@@
 					(unit 1)
 				)
-				(path "/0cf42e13-7c72-4f5f-898b-a3f851b94890/00000000-0000-0000-0000-00005c7c62ae"
-					(reference "Q?")
-					(unit 1)
-				)
 			)
 		)
@@
 					(unit 1)
 				)
-				(path "/0cf42e13-7c72-4f5f-898b-a3f851b94890/00000000-0000-0000-0000-00005c7c62ae"
-					(reference "Q?")
-					(unit 1)
-				)
 			)
 		)
@@
 					(unit 1)
 				)
-				(path "/0cf42e13-7c72-4f5f-898b-a3f851b94890/00000000-0000-0000-0000-00005c7c62ae"
-					(reference "#PWR?")
-					(unit 1)
-				)
 			)
 		)
@@
 					(unit 1)
 				)
-				(path "/0cf42e13-7c72-4f5f-898b-a3f851b94890/00000000-0000-0000-0000-00005c7c62ae"
-					(reference "#PWR?")
-					(unit 1)
-				)
 			)
 		)
@@
 					(unit 1)
 				)
-				(path "/0cf42e13-7c72-4f5f-898b-a3f851b94890/00000000-0000-0000-0000-00005c7c62ae"
-					(reference "#PWR?")
-					(unit 1)
-				)
 			)
 		)
@@
 					(unit 1)
 				)
-				(path "/0cf42e13-7c72-4f5f-898b-a3f851b94890/00000000-0000-0000-0000-00005c7c62ae"
-					(reference "R?")
-					(unit 1)
-				)
 			)
 		)
@@
 					(unit 1)
 				)
-				(path "/0cf42e13-7c72-4f5f-898b-a3f851b94890/00000000-0000-0000-0000-00005c7c62ae"
-					(reference "R?")
-					(unit 1)
-				)
 			)
 		)
@@
 					(unit 1)
 				)
-				(path "/0cf42e13-7c72-4f5f-898b-a3f851b94890/00000000-0000-0000-0000-00005c7c62ae"
-					(reference "R?")
-					(unit 1)
-				)
 			)
 		)
@@
 					(unit 1)
 				)
-				(path "/0cf42e13-7c72-4f5f-898b-a3f851b94890/00000000-0000-0000-0000-00005c7c62ae"
-					(reference "D?")
-					(unit 1)
-				)
 			)
 		)
@@
 					(unit 1)
 				)
-				(path "/0cf42e13-7c72-4f5f-898b-a3f851b94890/00000000-0000-0000-0000-00005c7c62ae"
-					(reference "R?")
-					(unit 1)
-				)
 			)
 		)
@@
 					(unit 1)
 				)
-				(path "/0cf42e13-7c72-4f5f-898b-a3f851b94890/00000000-0000-0000-0000-00005c7c62ae"
-					(reference "R?")
-					(unit 1)
-				)
 			)
 		)
@@
 					(unit 1)
 				)
-				(path "/0cf42e13-7c72-4f5f-898b-a3f851b94890/00000000-0000-0000-0000-00005c7c62ae"
-					(reference "R?")
-					(unit 1)
-				)
 			)
 		)
@@
 					(unit 1)
 				)
-				(path "/0cf42e13-7c72-4f5f-898b-a3f851b94890/00000000-0000-0000-0000-00005c7c62ae"
-					(reference "C?")
-					(unit 1)
-				)
 			)
 		)
@@
 					(unit 1)
 				)
-				(path "/0cf42e13-7c72-4f5f-898b-a3f851b94890/00000000-0000-0000-0000-00005c7c62ae"
-					(reference "#PWR?")
-					(unit 1)
-				)
 			)
 		)
@@
 					(unit 1)
 				)
-				(path "/0cf42e13-7c72-4f5f-898b-a3f851b94890/00000000-0000-0000-0000-00005c7c62ae"
-					(reference "#PWR?")
-					(unit 1)
-				)
 			)
 		)
@@
 					(unit 1)
 				)
-				(path "/0cf42e13-7c72-4f5f-898b-a3f851b94890/00000000-0000-0000-0000-00005c7c62ae"
-					(reference "Q?")
-					(unit 1)
-				)
 			)
 		)
@@
 					(unit 1)
 				)
-				(path "/0cf42e13-7c72-4f5f-898b-a3f851b94890/00000000-0000-0000-0000-00005c7c62ae"
-					(reference "Q?")
-					(unit 1)
-				)
 			)
 		)
@@
 					(unit 1)
 				)
-				(path "/0cf42e13-7c72-4f5f-898b-a3f851b94890/00000000-0000-0000-0000-00005c7c62ae"
-					(reference "Q?")
-					(unit 1)
-				)
 			)
 		)
@@
 					(unit 1)
 				)
-				(path "/0cf42e13-7c72-4f5f-898b-a3f851b94890/00000000-0000-0000-0000-00005c7c62ae"
-					(reference "#PWR?")
-					(unit 1)
-				)
 			)
 		)
@@
 					(unit 1)
 				)
-				(path "/0cf42e13-7c72-4f5f-898b-a3f851b94890/00000000-0000-0000-0000-00005c7c62ae"
-					(reference "#PWR?")
-					(unit 1)
-				)
 			)
 		)
@@
 					(unit 1)
 				)
-				(path "/0cf42e13-7c72-4f5f-898b-a3f851b94890/00000000-0000-0000-0000-00005c7c62ae"
-					(reference "#PWR?")
-					(unit 1)
-				)
 			)
 		)
@@
 					(unit 1)
 				)
-				(path "/0cf42e13-7c72-4f5f-898b-a3f851b94890/00000000-0000-0000-0000-00005c7c62ae"
-					(reference "R?")
-					(unit 1)
-				)
 			)
 		)
@@
 					(unit 1)
 				)
-				(path "/0cf42e13-7c72-4f5f-898b-a3f851b94890/00000000-0000-0000-0000-00005c7c62ae"
-					(reference "R?")
-					(unit 1)
-				)
 			)
 		)
@@
 					(unit 1)
 				)
-				(path "/0cf42e13-7c72-4f5f-898b-a3f851b94890/00000000-0000-0000-0000-00005c7c62ae"
-					(reference "R?")
-					(unit 1)
-				)
 			)
 		)
@@
 					(unit 1)
 				)
-				(path "/0cf42e13-7c72-4f5f-898b-a3f851b94890/00000000-0000-0000-0000-00005c7c62ae"
-					(reference "D?")
-					(unit 1)
-				)
 			)
 		)
@@
 					(unit 1)
 				)
-				(path "/0cf42e13-7c72-4f5f-898b-a3f851b94890/00000000-0000-0000-0000-00005c7c62ae"
-					(reference "R?")
-					(unit 1)
-				)
 			)
 		)
@@
 					(unit 1)
 				)
-				(path "/0cf42e13-7c72-4f5f-898b-a3f851b94890/00000000-0000-0000-0000-00005c7c62ae"
-					(reference "R?")
-					(unit 1)
-				)
 			)
 		)
@@
 					(unit 1)
 				)
-				(path "/0cf42e13-7c72-4f5f-898b-a3f851b94890/00000000-0000-0000-0000-00005c7c62ae"
-					(reference "R?")
-					(unit 1)
-				)
 			)
 		)
@@
 					(unit 1)
 				)
-				(path "/0cf42e13-7c72-4f5f-898b-a3f851b94890/00000000-0000-0000-0000-00005c7c62ae"
-					(reference "C?")
-					(unit 1)
-				)
 			)
 		)
@@
 					(unit 1)
 				)
-				(path "/0cf42e13-7c72-4f5f-898b-a3f851b94890/00000000-0000-0000-0000-00005c7c62ae"
-					(reference "C?")
-					(unit 1)
-				)
 			)
 		)
@@
 					(unit 1)
 				)
-				(path "/0cf42e13-7c72-4f5f-898b-a3f851b94890/00000000-0000-0000-0000-00005c7c62ae"
-					(reference "C?")
-					(unit 1)
-				)
 			)
 		)
@@
 					(unit 1)
 				)
-				(path "/0cf42e13-7c72-4f5f-898b-a3f851b94890/00000000-0000-0000-0000-00005c7c62ae"
-					(reference "C?")
-					(unit 1)
-				)
 			)
 		)
@@
 					(unit 1)
 				)
-				(path "/0cf42e13-7c72-4f5f-898b-a3f851b94890/00000000-0000-0000-0000-00005c7c62ae"
-					(reference "C?")
-					(unit 1)
-				)
 			)
 		)
@@
 					(unit 1)
 				)
-				(path "/0cf42e13-7c72-4f5f-898b-a3f851b94890/00000000-0000-0000-0000-00005c7c62ae"
-					(reference "C?")
-					(unit 1)
-				)
 			)
 		)
@@
 					(unit 1)
 				)
-				(path "/0cf42e13-7c72-4f5f-898b-a3f851b94890/00000000-0000-0000-0000-00005c7c62ae"
-					(reference "C?")
-					(unit 1)
-				)
 			)
 		)
@@
 					(unit 1)
 				)
-				(path "/0cf42e13-7c72-4f5f-898b-a3f851b94890/00000000-0000-0000-0000-00005c7c62ae"
-					(reference "#PWR?")
-					(unit 1)
-				)
 			)
 		)
@@
 					(unit 1)
 				)
-				(path "/0cf42e13-7c72-4f5f-898b-a3f851b94890/00000000-0000-0000-0000-00005c7c62ae"
-					(reference "#PWR?")
-					(unit 1)
-				)
 			)
 		)
@@
 					(unit 1)
 				)
-				(path "/0cf42e13-7c72-4f5f-898b-a3f851b94890/00000000-0000-0000-0000-00005c7c62ae"
-					(reference "#PWR?")
-					(unit 1)
-				)
 			)
 		)
@@
 					(unit 1)
 				)
-				(path "/0cf42e13-7c72-4f5f-898b-a3f851b94890/00000000-0000-0000-0000-00005c7c62ae"
-					(reference "#PWR?")
-					(unit 1)
-				)
 			)
 		)
@@
 					(unit 1)
 				)
-				(path "/0cf42e13-7c72-4f5f-898b-a3f851b94890/00000000-0000-0000-0000-00005852a88e"
-					(reference "R?")
-					(unit 1)
-				)
-				(path "/0cf42e13-7c72-4f5f-898b-a3f851b94890/00000000-0000-0000-0000-00005c7c62ae"
-					(reference "R?")
-					(unit 1)
-				)

Commit message: [+] complete PCB design
Changed lines of the file:
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@@
 	)
 	(junction
+		(at 200.66 154.94)
+		(diameter 0)
+		(color 0 0 0 0)
+	)
+	(junction
 		(at 100.33 138.43)
 		(diameter 0)
@@
 	)
 	(junction
+		(at 200.66 168.91)
+		(diameter 0)
+		(color 0 0 0 0)
+	)
+	(junction
 		(at 254 71.12)
 		(diameter 0)
@@
 					(unit 1)
 				)
+			)
+		)
+	)
+	(symbol
+		(lib_id "DFTBoard-rescue:PWR_FLAG")
+		(at 200.66 154.94 90)
+		(unit 1)
+		(exclude_from_sim no)
+		(in_bom yes)
+		(on_board yes)
+		(dnp no)
+		(property "Reference" "#FLG0802"
+			(at 198.755 154.94 0)
+			(effects
+				(font
+					(size 1.27 1.27)
+				)
+				(hide yes)
+			)
+		)
+		(property "Value" "PWR_FLAG"
+			(at 197.4088 154.94 90)
+			(effects
+				(font
+					(size 1.27 1.27)
+				)
+				(justify left)
+			)
+		)
+		(property "Footprint" ""
+			(at 200.66 154.94 0)
+			(effects
+				(font
+					(size 1.27 1.27)
+				)
+				(hide yes)
+			)
+		)
+		(property "Datasheet" ""
+			(at 200.66 154.94 0)
+			(effects
+				(font
+					(size 1.27 1.27)
+				)
+				(hide yes)
+			)
+		)
+		(property "Description" ""
+			(at 200.66 154.94 0)
+			(effects
+				(font
+					(size 1.27 1.27)
+				)
+				(hide yes)
+			)
+		)
+		(pin "1"
+		)
+		(instances
+			(project "DFTBoard"
+				(path "/0cf42e13-7c72-4f5f-898b-a3f851b94890/00000000-0000-0000-0000-000058508444"
+					(reference "#FLG0802")
+					(unit 1)
+				)
+			)
+		)
+	)
+	(symbol
+		(lib_id "DFTBoard-rescue:PWR_FLAG")
+		(at 200.66 168.91 90)
+		(unit 1)
+		(exclude_from_sim no)
+		(in_bom yes)
+		(on_board yes)
+		(dnp no)
+		(property "Reference" "#FLG0801"
+			(at 198.755 168.91 0)
+			(effects
+				(font
+					(size 1.27 1.27)
+				)
+				(hide yes)
+			)
+		)
+		(property "Value" "PWR_FLAG"
+			(at 197.4088 168.91 90)
+			(effects
+				(font
+					(size 1.27 1.27)
+				)
+				(justify left)
+			)
+		)
+		(property "Footprint" ""
+			(at 200.66 168.91 0)
+			(effects
+				(font
+					(size 1.27 1.27)
+				)
+				(hide yes)
+			)
+		)
+		(property "Datasheet" ""
+			(at 200.66 168.91 0)
+			(effects
+				(font
+					(size 1.27 1.27)
+				)
+				(hide yes)
+			)
+		)
+		(property "Description" ""
+			(at 200.66 168.91 0)
+			(effects
+				(font
+					(size 1.27 1.27)
+				)
+				(hide yes)
+			)
+		)
+		(pin "1"
+		)
+		(instances
+			(project "DFTBoard"
+				(path "/0cf42e13-7c72-4f5f-898b-a3f851b94890/00000000-0000-0000-0000-000058508444"
+					(reference "#FLG0801")
+					(unit 1)
+				)

Commit message: [+] add xdc files
Parts:
- removed C43, C44: 1uF, Capacitor_SMD:C_0402_1005Metric, symbol Device:C
- removed D1, D2: LED_RGB, DFTcustom:PLCC6-SM-RGB-LED, symbol DFTBoard-rescue:LED_RGB-RESCUE-DFTBoard-
- removed Q1, Q2, Q3, Q4, Q5, Q6: IRLML2502, Package_TO_SOT_SMD:SOT-23, symbol DFTBoard-rescue:IRLML2502-
- removed R11, R12, R13, R14, R15, R16, R19, R20, R22, R23: 100, Resistor_SMD:R_0402_1005Metric, symbol Device:R
- removed R21, R24: 150, Resistor_SMD:R_0402_1005Metric, symbol Device:R
