File: PCB/LCD50.kicad_sch (KiCad schematic)
At the start: 33 parts, among them J701 FFC2B28-40-G, J702 Conn_01x06_Female, SW701 SW_PUSH, SW702 SW_PUSH, SW703 SW_PUSH, SW704 SW_PUSH, U20 xc7z020clg484, U701 MT3608

Commit message: some changes
Connections:
- net JOYCS: no longer U20.AB4 (IO_L16N_T2_13)
- net JOYMISO: no longer U20.AB6 (IO_L17N_T2_13)
- net JOYMOSI: no longer U20.AB5 (IO_L16P_T2_13)
- net JOYSCK: no longer U20.AB7 (IO_L17P_T2_13)
- no-connect marks 20 -> 24
Changed lines of the file:
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@@
 	)
 	(no_connect
+		(at 163.83 130.81)
+	)
+	(no_connect
 		(at 92.71 130.175)
 	)
@@
 	)
 	(no_connect
+		(at 163.83 133.35)
+	)
+	(no_connect
 		(at 163.83 151.13)
 	)
@@
 	)
 	(no_connect
+		(at 163.83 128.27)
+	)
+	(no_connect
 		(at 163.83 44.45)
 	)
 	(no_connect
+		(at 163.83 125.73)
+	)
+	(no_connect
 		(at 163.83 148.59)
 	)
@@
 	(wire
 		(pts
-			(xy 151.765 125.73) (xy 163.83 125.73)
-		)
-		(stroke
-			(width 0)
-			(type default)
-		)
-	)
-	(wire
-		(pts
 			(xy 85.725 74.295) (xy 92.71 74.295)
 		)
@@
 	(wire
 		(pts
-			(xy 73.025 167.005) (xy 85.09 167.005)
-		)
-		(stroke
-			(width 0)
-			(type default)
-		)
-	)
-	(wire
-		(pts
 			(xy 73.025 174.625) (xy 85.09 174.625)
 		)
@@
 	(wire
 		(pts
-			(xy 151.765 133.35) (xy 163.83 133.35)
-		)
-		(stroke
-			(width 0)
-			(type default)
-		)
-	)
-	(wire
-		(pts
 			(xy 155.575 52.07) (xy 163.83 52.07)
 		)
@@
 		)
 	)
-	(wire
-		(pts
-			(xy 151.765 130.81) (xy 163.83 130.81)
-		)
-		(stroke
-			(width 0)
-			(type default)
-		)
-	)
 	(bus
 		(pts
@@
 		)
 	)
+	(wire
+		(pts
+			(xy 73.025 167.005) (xy 85.09 167.005)
+		)
+		(stroke
+			(width 0)
+			(type default)
+		)
+	)
 	(bus
 		(pts
@@
 	(wire
 		(pts
-			(xy 151.765 128.27) (xy 163.83 128.27)
-		)
-		(stroke
-			(width 0)
-			(type default)
-		)
-	)
-	(wire
-		(pts
 			(xy 189.23 176.53) (xy 189.23 179.07)
 		)
@@
 		)
 	)
-	(label "JOYSCK"
-		(at 73.025 174.625 0)
-		(fields_autoplaced yes)
-		(effects
-			(font
-				(size 1.27 1.27)
-			)
-			(justify left bottom)
-		)
-	)
 	(label "LCDGREEN5"
 		(at 163.83 82.55 0)
@@
 		)
 	)
-	(label "JOYMISO"
-		(at 151.765 130.81 0)
-		(fields_autoplaced yes)
-		(effects
-			(font
-				(size 1.27 1.27)
-			)
-			(justify left bottom)
-		)
-	)
 	(label "LCDBLUE1"
 		(at 92.71 97.155 0)
@@
 		)
 	)
-	(label "JOYSCK"
-		(at 151.765 133.35 0)
-		(fields_autoplaced yes)
-		(effects
-			(font
-				(size 1.27 1.27)
-			)
-			(justify left bottom)
-		)
-	)
 	(label "LCDRED3"
 		(at 92.71 61.595 0)
@@
 		)
 	)
-	(label "JOYMOSI"
-		(at 151.765 128.27 0)
-		(fields_autoplaced yes)
-		(effects
-			(font
-				(size 1.27 1.27)
-			)
-			(justify left bottom)
-		)
-	)
 	(label "LCDGREEN0"
 		(at 163.83 69.85 0)
@@
 		)
 	)
-	(label "JOYCS"
-		(at 73.025 167.005 0)
-		(fields_autoplaced yes)
-		(effects
-			(font
-				(size 1.27 1.27)
-			)
-			(justify left bottom)
-		)
-	)
 	(label "LCDGREEN2"
 		(at 163.83 74.93 0)
@@
 		)
 	)
-	(label "JOYMOSI"
-		(at 73.025 169.545 0)
-		(fields_autoplaced yes)
-		(effects
-			(font
-				(size 1.27 1.27)
-			)
-			(justify left bottom)
-		)
-	)
 	(label "LCDBLUE6"
 		(at 163.83 105.41 0)
@@
 		)
 	)
-	(label "JOYMISO"
-		(at 73.025 172.085 0)
-		(fields_autoplaced yes)
-		(effects
-			(font
-				(size 1.27 1.27)
-			)
-			(justify left bottom)
-		)
-	)
 	(label "LCDDHSYNC"
 		(at 142.875 115.57 0)
@@
 		)
 	)
-	(label "JOYCS"
-		(at 151.765 125.73 0)
-		(fields_autoplaced yes)
-		(effects
-			(font
-				(size 1.27 1.27)
-			)
-			(justify left bottom)
-		)
-	)
 	(label "LCDRED6"
 		(at 163.83 64.77 0)
@@
 		)
 	)
+	(global_label "JOYCS"
+		(shape input)
+		(at 73.025 167.005 180)
+		(fields_autoplaced yes)
+		(effects
+			(font
+				(size 1.27 1.27)
+			)
+			(justify right)
+		)
+		(property "Intersheetrefs" "${INTERSHEET_REFS}"
+			(at 64.8278 167.005 0)
+			(effects
+				(font
+					(size 1.27 1.27)
+				)
+				(justify right)
+				(hide yes)
+			)
+		)
+	)
 	(global_label "LCDGREEN[0..7]"
 		(shape input)
@@
 		)
 	)
+	(global_label "JOYSCK"
+		(shape input)
+		(at 73.025 174.625 180)
+		(fields_autoplaced yes)
+		(effects
+			(font
+				(size 1.27 1.27)
+			)
+			(justify right)
+		)
+		(property "Intersheetrefs" "${INTERSHEET_REFS}"
+			(at 63.5578 174.625 0)
+			(effects
+				(font
+					(size 1.27 1.27)
+				)
+				(justify right)
+				(hide yes)
+			)
+		)
+	)
 	(global_label "BTN1"
 		(shape bidirectional)
@@
 		)
 	)
+	(global_label "JOYMOSI"
+		(shape input)
+		(at 73.025 169.545 180)
+		(fields_autoplaced yes)
+		(effects
+			(font
+				(size 1.27 1.27)
+			)
+			(justify right)
+		)
+		(property "Intersheetrefs" "${INTERSHEET_REFS}"
+			(at 62.7111 169.545 0)
+			(effects
+				(font
+					(size 1.27 1.27)
+				)
+				(justify right)
+				(hide yes)
+			)
+		)
+	)
 	(global_label "LCDBLUE[0..7]"
 		(shape input)
@@
 				(hide yes)
 			)
+		)
+	)
+	(global_label "JOYMISO"
+		(shape input)
+		(at 73.025 172.085 180)
+		(fields_autoplaced yes)
+		(effects
+			(font
+				(size 1.27 1.27)
+			)
+			(justify right)
+		)
+		(property "Intersheetrefs" "${INTERSHEET_REFS}"
+			(at 62.7111 172.085 0)
+			(effects
+				(font
+					(size 1.27 1.27)
+				)
+				(justify right)
+				(hide yes)
+			)

Commit message: [+] Layouting
Parts:
- J702: footprint Connector_PinHeader_1.00mm:PinHeader_1x06_P1.00mm_Vertical_SMD_Pin1Right -> Connector_PinSocket_2.54mm:PinSocket_1x06_P2.54mm_Horizontal
Other:
- moved on the sheet: U20E
