File: PCB/Power_management.kicad_sch (KiCad schematic)
At the start: 114 parts, among them J401 PJ-037AH, Q401 2N7002E, Q402 PMBT3904YS, Q403 2N3906, Q404 2N7002E, Q405 2N7002E, Q406 AP2307GN, Q407 2N3906, SW401 SW_Wuerth_450301014042, U401 TPS65400RGZR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

Commit message: merge commit
Connections:
- net GND: now also C440.2, C441.2
Changed lines of the file:
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@@
 	)
 	(junction
+		(at 306.07 186.69)
+		(diameter 0)
+		(color 0 0 0 0)
+	)
+	(junction
 		(at 466.09 138.43)
 		(diameter 0)
@@
 	(wire
 		(pts
+			(xy 306.07 186.69) (xy 306.705 186.69)
+		)
+		(stroke
+			(width 0)
+			(type default)
+		)
+	)
+	(wire
+		(pts
 			(xy 473.075 184.785) (xy 473.075 187.325)
 		)
@@
 	(wire
 		(pts
-			(xy 300.99 186.69) (xy 306.705 186.69)
+			(xy 300.99 186.69) (xy 306.07 186.69)
 		)
 		(stroke
@@
 	(symbol
 		(lib_id "Device:C_Small")
-		(at 306.705 189.23 0)
+		(at 306.07 189.23 0)
 		(unit 1)
 		(exclude_from_sim no)
@@
 		(dnp no)
 		(property "Reference" "C441"
-			(at 309.88 189.2362 0)
+			(at 309.245 189.2362 0)
 			(effects
 				(font
@@
 		)
 		(property "Value" "22uF 25V 0805"
-			(at 309.88 190.5062 0)
+			(at 309.245 190.5062 0)
 			(effects
 				(font
@@
 		)
 		(property "Footprint" "Capacitor_SMD:C_0805_2012Metric"
-			(at 306.705 189.23 0)
+			(at 306.07 189.23 0)
 			(effects
 				(font
@@
 		)
 		(property "Datasheet" "~"
-			(at 306.705 189.23 0)
+			(at 306.07 189.23 0)
 			(effects
 				(font
@@
 		)
 		(property "Description" "Unpolarized capacitor, small symbol"
-			(at 306.705 189.23 0)
+			(at 306.07 189.23 0)
 			(effects
 				(font
@@
 	)
 	(symbol
+		(lib_id "power:GND")
+		(at 300.99 191.77 0)
+		(unit 1)
+		(exclude_from_sim no)
+		(in_bom yes)
+		(on_board yes)
+		(dnp no)
+		(fields_autoplaced yes)
+		(property "Reference" "#PWR01"
+			(at 300.99 198.12 0)
+			(effects
+				(font
+					(size 1.27 1.27)
+				)
+				(hide yes)
+			)
+		)
+		(property "Value" "GND"
+			(at 300.99 196.85 0)
+			(effects
+				(font
+					(size 1.27 1.27)
+				)
+			)
+		)
+		(property "Footprint" ""
+			(at 300.99 191.77 0)
+			(effects
+				(font
+					(size 1.27 1.27)
+				)
+				(hide yes)
+			)
+		)
+		(property "Datasheet" ""
+			(at 300.99 191.77 0)
+			(effects
+				(font
+					(size 1.27 1.27)
+				)
+				(hide yes)
+			)
+		)
+		(property "Description" "Power symbol creates a global label with name \"GND\" , ground"
+			(at 300.99 191.77 0)
+			(effects
+				(font
+					(size 1.27 1.27)
+				)
+				(hide yes)
+			)
+		)
+		(pin "1"
+		)
+		(instances
+			(project "gameboy"
+				(path "/bfbf29d7-ad29-43e7-b23f-5805508cd3f0/a40e8631-6af3-4d0f-b1b9-51a13e66bfc2"
+					(reference "#PWR01")
+					(unit 1)
+				)
+			)
+		)
+	)
+	(symbol
 		(lib_id "Transistor_FET:2N7002E")
 		(at 256.54 220.345 0)
@@
 					(unit 1)
 				)
+			)
+		)
+	)
+	(symbol
+		(lib_id "power:GND")
+		(at 306.07 191.77 0)
+		(unit 1)
+		(exclude_from_sim no)
+		(in_bom yes)
+		(on_board yes)
+		(dnp no)
+		(fields_autoplaced yes)
+		(property "Reference" "#PWR02"
+			(at 306.07 198.12 0)
+			(effects
+				(font
+					(size 1.27 1.27)
+				)
+				(hide yes)
+			)
+		)
+		(property "Value" "GND"
+			(at 306.07 196.85 0)
+			(effects
+				(font
+					(size 1.27 1.27)
+				)
+			)
+		)
+		(property "Footprint" ""
+			(at 306.07 191.77 0)
+			(effects
+				(font
+					(size 1.27 1.27)
+				)
+				(hide yes)
+			)
+		)
+		(property "Datasheet" ""
+			(at 306.07 191.77 0)
+			(effects
+				(font
+					(size 1.27 1.27)
+				)
+				(hide yes)
+			)
+		)
+		(property "Description" "Power symbol creates a global label with name \"GND\" , ground"
+			(at 306.07 191.77 0)
+			(effects
+				(font
+					(size 1.27 1.27)
+				)
+				(hide yes)
+			)
+		)
+		(pin "1"
+		)
+		(instances
+			(project "gameboy"
+				(path "/bfbf29d7-ad29-43e7-b23f-5805508cd3f0/a40e8631-6af3-4d0f-b1b9-51a13e66bfc2"
+					(reference "#PWR02")
+					(unit 1)
+				)
