File: PCB/Storage.kicad_sch (KiCad schematic)
At the start: 24 parts, among them J601 Micro_SD_Card_Det, U17 FTDITypeUART, U18 ABRACON-ASDMB, U20 xc7z020clg484

Commit message: [+] routing done, need to fix minor errors.
Parts:
- gave numbers to parts that had none: 18
